File: interface2_cartridge.sch (KiCad schematic (older format))
At the start: 13 parts, among them J1 cartridge_IF2, J2 Conn_01x05, U1 29F010-TSOP-SP

Commit message: final design
Parts:
- U1: value 29F010-TSOP-SP -> AM29F010B; footprint Package_LCC:PLCC-32 -> SINCLAIR:PLCC-32; symbol Memory_Flash:29F010-TSOP-SP -> Memory_EPROM:27C010
Connections:
- wire segments 94 -> 98
- no-connect marks 0 -> 1
